Commit message: diff drive and manipulator work

File: turtlebot3_manipulation_description/gazebo/turtlebot3_waffle_pi.gazebo.xacro (robot description, xacro)
@@ -6,146 +6,189 @@
 <robot xmlns:xacro="http://ros.org/wiki/xacro">
   <xacro:macro name="turtlebot3_waffle_pi_gazebo" params="prefix">
-  <xacro:property name="laser_visual"  value="true"/>
-  <xacro:property name="camera_visual" value="true"/>
-  <xacro:property name="imu_visual"    value="true"/>
-  <gazebo reference="${prefix}base_link">
-    <material>Gazebo/DarkGrey</material>
-  </gazebo>
-  <gazebo reference="${prefix}wheel_left_link">
-    <mu1>10000</mu1>
-    <mu2>10000</mu2>
-    <kp>500000.0</kp>
-    <kd>10.0</kd>
-    <minDepth>0.001</minDepth>
-    <maxVel>0.1</maxVel>
-    <fdir1>1 0 0</fdir1>
-    <material>Gazebo/FlatBlack</material>
-  </gazebo>
-  <gazebo reference="${prefix}wheel_right_link">
-    <mu1>10000</mu1>
-    <mu2>10000</mu2>
-    <kp>500000.0</kp>
-    <kd>10.0</kd>
-    <minDepth>0.001</minDepth>
-    <maxVel>0.1</maxVel>
-    <fdir1>1 0 0</fdir1>
-    <material>Gazebo/FlatBlack</material>
-  </gazebo>
-  <gazebo reference="${prefix}caster_back_right_link">
-    <mu1>0.1</mu1>
-    <mu2>0.1</mu2>
-    <kp>1000000.0</kp>
-    <kd>100.0</kd>
-    <minDepth>0.001</minDepth>
-    <maxVel>1.0</maxVel>
-    <material>Gazebo/FlatBlack</material>
-  </gazebo>
-  <gazebo reference="${prefix}caster_back_left_link">
-    <mu1>0.1</mu1>
-    <mu2>0.1</mu2>
-    <kp>1000000.0</kp>
-    <kd>100.0</kd>
-    <minDepth>0.001</minDepth>
-    <maxVel>1.0</maxVel>
-    <material>Gazebo/FlatBlack</material>
-  </gazebo>
-  <gazebo reference="${prefix}imu_link">
-    <material>Gazebo/Grey</material>
-    <sensor type="imu" name="imu">
-      <always_on>true</always_on>
-      <update_rate>100.0</update_rate>
-      <visualize>${imu_visual}</visualize>
-    </sensor>
-  </gazebo>
-  <gazebo>
-    <plugin name='diff_drive' filename='libgazebo_ros_diff_drive.so'>
-      <ros>
-        <namespace></namespace>
-        <remapping>cmd_vel:=cmd_vel</remapping>
-        <remapping>odom:=odom</remapping>
-      </ros>
-      <left_joint>wheel_left_joint</left_joint>
-      <right_joint>wheel_right_joint</right_joint>
-      <wheel_separation>0.287</wheel_separation>
-      <wheel_diameter>0.066</wheel_diameter>
-      <max_wheel_torque>20</max_wheel_torque>
-      <max_wheel_acceleration>1.0</max_wheel_acceleration>
-      <publish_odom>true</publish_odom>
-      <publish_odom_tf>true</publish_odom_tf>
-      <publish_wheel_tf>false</publish_wheel_tf>
-      <odometry_frame>odom</odometry_frame>
-      <robot_base_frame>base_footprint</robot_base_frame>
-    </plugin>
-  </gazebo>
-  <gazebo reference="${prefix}base_scan">
-    <material>Gazebo/FlatBlack</material>
-    <sensor type="ray" name="lds_lfcd_sensor">
-      <pose>0 0 0 0 0 0</pose>
-      <always_on>true</always_on>
-      <update_rate>5.0</update_rate>
-      <visualize>${laser_visual}</visualize>
-      <ray>
-        <scan>
-          <horizontal>
-            <samples>360</samples>
-            <resolution>1</resolution>
-            <min_angle>0.0</min_angle>
-            <max_angle>6.28319</max_angle>
-          </horizontal>
-        </scan>
-        <range>
-          <min>0.120</min>
-          <max>3.5</max>
-          <resolution>0.015</resolution>
-        </range>
-        <noise>
-          <type>gaussian</type>
-          <mean>0.0</mean>
-          <stddev>0.01</stddev>
-        </noise>
-      </ray>
-      <plugin name="gazebo_ros_lds_lfcd_controller" filename="libgazebo_ros_ray_sensor.so">
-        <ros>
-          <namespace></namespace>
-          <remapping>~/out:=scan</remapping>
-        </ros>
-        <output_type>sensor_msgs/LaserScan</output_type>
+    <xacro:property name="laser_visual" value="true" />
+    <xacro:property name="camera_visual" value="true" />
+    <xacro:property name="imu_visual" value="true" />
+    <xacro:macro name="ray_sensor"
+      params="sensor_name gazebo update_rate visualize
+            h_samples h_res h_min_angle h_max_angle
+            r_min r_max r_res *plugin">
+      <sensor name="${sensor_name}" type="gpu_lidar">
+        <update_rate>${update_rate}</update_rate>
+        <visualize>${visualize}</visualize>
+        <always_on>true</always_on>
+        <!-- <gz_frame_id>${sensor_name}_link</gz_frame_id> -->
+        <gz_frame_id>${prefix}base_scan</gz_frame_id>
+        <topic>scan</topic>
+        <lidar>
+          <scan>
+            <horizontal>
+              <samples>${h_samples}</samples>
+              <resolution>${h_res}</resolution>
+              <min_angle>${h_min_angle}</min_angle>
+              <max_angle>${h_max_angle}</max_angle>
+            </horizontal>
+          </scan>
+          <range>
+            <min>${r_min}</min>
+            <max>${r_max}</max>
+            <resolution>${r_res}</resolution>
+          </range>
+        </lidar>
+      </sensor>
+    </xacro:macro>
+    <gazebo reference="${prefix}base_link">
+      <material>Gazebo/DarkGrey</material>
+    </gazebo>
+    <gazebo reference="${prefix}wheel_left_link">
+      <mu1>10000</mu1>
+      <mu2>10000</mu2>
+      <kp>500000.0</kp>
+      <kd>10.0</kd>
+      <minDepth>0.001</minDepth>
+      <maxVel>0.1</maxVel>
+      <fdir1>1 0 0</fdir1>
+      <material>Gazebo/FlatBlack</material>
+    </gazebo>
+    <gazebo reference="${prefix}wheel_right_link">
+      <mu1>10000</mu1>
+      <mu2>10000</mu2>
+      <kp>500000.0</kp>
+      <kd>10.0</kd>
+      <minDepth>0.001</minDepth>
+      <maxVel>0.1</maxVel>
+      <fdir1>1 0 0</fdir1>
+      <material>Gazebo/FlatBlack</material>
+    </gazebo>
+    <gazebo reference="${prefix}caster_back_right_link">
+      <mu1>0.1</mu1>
+      <mu2>0.1</mu2>
+      <kp>1000000.0</kp>
+      <kd>100.0</kd>
+      <minDepth>0.001</minDepth>
+      <maxVel>1.0</maxVel>
+      <material>Gazebo/FlatBlack</material>
+    </gazebo>
+    <gazebo reference="${prefix}caster_back_left_link">
+      <mu1>0.1</mu1>
+      <mu2>0.1</mu2>
+      <kp>1000000.0</kp>
+      <kd>100.0</kd>
+      <minDepth>0.001</minDepth>
+      <maxVel>1.0</maxVel>
+      <material>Gazebo/FlatBlack</material>
+    </gazebo>
+    <gazebo reference="${prefix}imu_link">
+      <material>Gazebo/Grey</material>
+      <sensor type="imu" name="imu">
+        <always_on>true</always_on>
+        <update_rate>100</update_rate>
+        <topic>imu</topic>
+        <imu>
+          <angular_velocity>
+            <x>
+              <noise type="gaussian">
+                <mean>0.0</mean>
+                <stddev>2e-4</stddev>
+              </noise>
+            </x>
+            <y>
+              <noise type="gaussian">
+                <mean>0.0</mean>
+                <stddev>2e-4</stddev>
+              </noise>
+            </y>
+            <z>
+              <noise type="gaussian">
+                <mean>0.0</mean>
+                <stddev>2e-4</stddev>
+              </noise>
+            </z>
+          </angular_velocity>
+          <linear_acceleration>
+            <x>
+              <noise type="gaussian">
+                <mean>0.0</mean>
+                <stddev>2e-4</stddev>
+              </noise>
+            </x>
+            <y>
+              <noise type="gaussian">
+                <mean>0.0</mean>
+                <stddev>2e-4</stddev>
+              </noise>
+            </y>
+            <z>
+              <noise type="gaussian">
+                <mean>0.0</mean>
+                <stddev>2e-4</stddev>
+              </noise>
+            </z>
+          </linear_acceleration>
+        </imu>
+      </sensor>
+    </gazebo>
+    <gazebo>
+      <plugin
+        filename="gz-sim-diff-drive-system"
+        name="gz::sim::systems::DiffDrive">
+        <left_joint>wheel_left_joint</left_joint>
+        <right_joint>wheel_right_joint</right_joint>
+        <wheel_separation>0.287</wheel_separation>
+        <wheel_radius>0.033</wheel_radius>
+        <max_linear_acceleration>2</max_linear_acceleration>
+        <min_linear_acceleration>-2</min_linear_acceleration>
+        <max_angular_acceleration>3</max_angular_acceleration>
+        <min_angular_acceleration>-3</min_angular_acceleration>
+        <max_linear_velocity>0.5</max_linear_velocity>
+        <min_linear_velocity>-0.5</min_linear_velocity>
+        <max_angular_velocity>2.0</max_angular_velocity>
+        <min_angular_velocity>-2.0</min_angular_velocity>
+        <topic>cmd_vel</topic>
+        <odom_topic>odom</odom_topic>
+        <tf_topic>tf</tf_topic>
+        <frame_id>odom</frame_id>
+        <child_frame_id>base_footprint</child_frame_id>
+        <odom_publish_frequency>30</odom_publish_frequency>
       </plugin>
-    </sensor>
-  </gazebo>
-  <gazebo reference="${prefix}camera_rgb_frame">
-    <sensor type="camera" name="pi_camera">
-      <update_rate>30</update_rate>
-      <always_on>true</always_on>
-      <visualize>${camera_visual}</visualize>
-      <camera>
-          <horizontal_fov>1.085595</horizontal_fov>
+      <plugin
+        filename="gz-sim-joint-state-publisher-system"
+        name="gz::sim::systems::JointStatePublisher">
+        <joint_name>wheel_left_joint</joint_name>
+        <joint_name>wheel_right_joint</joint_name>
+        <topic>joint_states</topic>
+        <update_rate>30</update_rate>
+      </plugin>
+    </gazebo>
+    <gazebo reference="${prefix}base_scan">
+      <xacro:ray_sensor sensor_name="scan" gazebo="ignition"
+        update_rate="10.0" visualize="true"
+        h_samples="360" h_res="1.0" h_min_angle="0.000" h_max_angle="6.280000"
+        r_min="0.164" r_max="20.0" r_res="0.01">
+        <plugin name="dummy" filename="dummyfile"></plugin>
+      </xacro:ray_sensor>
+      <!-- <xacro:material_darkgray /> -->
+      <material>Gazebo/DarkGrey</material>
+    </gazebo>
+    <gazebo reference="${prefix}camera_rgb_frame">
+      <sensor type="camera" name="pi_camera">
+        <always_on>1</always_on>
+        <camera>
+          <horizontal_fov>1.25</horizontal_fov>
           <image>
-              <width>640</width>
-              <height>480</height>
-              <format>R8G8B8</format>
+            <width>640</width>
+            <height>480</height>
           </image>
           <clip>
-              <near>0.03</near>
-              <far>100</far>
+            <near>0.3</near>
+            <far>100</far>
           </clip>
-          <noise>
-            <type>gaussian</type>
-            <!-- Noise is sampled independently per pixel on each frame.
-                 That pixel's noise value is added to each of its color
-                 channels, which at that point lie in the range [0,1]. -->
-            <mean>0.0</mean>
-            <stddev>0.007</stddev>
-          </noise>
-      </camera>
-      <plugin name="camera_controller" filename="libgazebo_ros_camera.so">
-        <ros>
-          <namespace></namespace>
-          <remapping>image_raw:=image_raw</remapping>
-          <remapping>camera_info:=camera_info</remapping>
-        </ros>
-      </plugin>
-    </sensor>
-  </gazebo>
+          <optical_frame_id>camera_rgb_optical_frame</optical_frame_id>
+        </camera>
+        <update_rate>10</update_rate>
+        <visualize>true</visualize>
+        <topic>image_raw</topic>
+      </sensor>
+      <material>Gazebo/DarkGrey</material>
+    </gazebo>
   </xacro:macro>
 </robot>

File: turtlebot3_manipulation_description/ros2_control/turtlebot3_manipulation_system.ros2_control.xacro (robot description, xacro)
@@ -10,5 +10,5 @@
       <xacro:if value="$(arg use_sim)">
         <hardware>
-          <plugin>gazebo_ros2_control/GazeboSystem</plugin>
+          <plugin>gz_ros2_control/GazeboSimSystem</plugin>
         </hardware>
       </xacro:if>

File: turtlebot3_manipulation_description/urdf/turtlebot3_manipulation.urdf.xacro (robot description, xacro)
@@ -22,7 +22,7 @@
   <!-- Used for fixing OpenManipulator-X on TurtleBot3 Waffle Pi -->
   <joint name="$(arg prefix)base_fixed" type="fixed">
-    <parent link="$(arg prefix)base_link"/>
-    <child link="$(arg prefix)link1"/>
-    <origin xyz="-0.092 0.0 0.091" rpy="0 0 0"/>
+    <parent link="$(arg prefix)base_link" />
+    <child link="$(arg prefix)link1" />
+    <origin xyz="-0.092 0.0 0.091" rpy="0 0 0" />
   </joint>
   <xacro:open_manipulator_x prefix="$(arg prefix)" />
@@ -31,8 +31,10 @@
     name="TurtleBot3ManipulationSystem" prefix="$(arg prefix)" use_sim="$(arg use_sim)"
     use_fake_hardware="$(arg use_fake_hardware)"
-    fake_sensor_commands="$(arg fake_sensor_commands)"/>
+    fake_sensor_commands="$(arg fake_sensor_commands)" />
   <gazebo>
-    <plugin name="gazebo_ros2_control" filename="libgazebo_ros2_control.so">
-      <parameters>$(find turtlebot3_manipulation_bringup)/config/gazebo_controller_manager.yaml</parameters>
+    <plugin filename="gz_ros2_control-system" name="gz_ros2_control::GazeboSimROS2ControlPlugin">
+      <robot_param>robot_description</robot_param>
+      <robot_param_node>robot_state_publisher</robot_param_node>
+      <parameters>$(find turtlebot3_manipulation_bringup)/config/hardware_controller_manager.yaml</parameters>
     </plugin>
   </gazebo>

Commit message: code for maze testing hw

File: turtlebot3_manipulation_description/gazebo/turtlebot3_waffle_pi.gazebo.xacro (robot description, xacro)
@@ -18,5 +18,5 @@
         <always_on>true</always_on>
         <!-- <gz_frame_id>${sensor_name}_link</gz_frame_id> -->
-        <gz_frame_id>${prefix}base_scan</gz_frame_id>
+        <!-- <gz_frame_id>${prefix}base_scan</gz_frame_id> -->
         <topic>scan</topic>
         <lidar>
@@ -170,4 +170,5 @@
       <material>Gazebo/DarkGrey</material>
     </gazebo>
+    <!--
     <gazebo reference="${prefix}camera_rgb_frame">
       <sensor type="camera" name="pi_camera">
@@ -190,4 +191,30 @@
       </sensor>
       <material>Gazebo/DarkGrey</material>
+    </gazebo> -->
+    <gazebo reference="${prefix}camera_rgb_frame">
+      <sensor type="camera" name="pi_camera">
+        <update_rate>30.0</update_rate>
+        <camera name="head">
+          <camera_info_topic>camera/camera_info</camera_info_topic>
+          <horizontal_fov>1.1519</horizontal_fov>
+          <image>
+            <width>640</width>
+            <height>480</height>
+            <format>R8G8B8</format>
+          </image>
+          <clip>
+            <near>0.02</near>
+            <far>300</far>
+          </clip>
+          <noise>
+            <type>gaussian</type>
+            <mean>0.0</mean>
+            <stddev>0.007</stddev>
+          </noise>
+        </camera>
+        <topic>camera/image_raw</topic>
+        <!-- <gz_frame_id>camera</gz_frame_id> -->
+      </sensor>
+      <material>Gazebo/DarkGrey</material>
     </gazebo>
   </xacro:macro>

File: turtlebot3_manipulation_description/urdf/turtlebot3_waffle_pi.urdf.xacro (robot description, xacro)
@@ -172,9 +172,8 @@
     <parent link="${prefix}base_link"/>
     <child link="${prefix}camera_link"/>
-    <origin xyz="0.073 -0.011 0.084" rpy="0 0 0"/>
+    <origin xyz="0.133 0.0 0.095" rpy="0 0 0"/>
   </joint>
   <link name="${prefix}camera_link">
     <collision>
-      <origin xyz="0.005 0.011 0.013" rpy="0 0 0"/>
       <geometry>
         <box size="0.015 0.030 0.027"/>
