Commit message: some cleanup and aligning with the upstream jazzy branch

File: turtlebot3_manipulation_description/urdf/turtlebot3_manipulation.urdf.xacro (robot description, xacro)
@@ -22,7 +22,7 @@
   <!-- Used for fixing OpenManipulator-X on TurtleBot3 Waffle Pi -->
   <joint name="$(arg prefix)base_fixed" type="fixed">
-    <parent link="$(arg prefix)base_link" />
-    <child link="$(arg prefix)link1" />
-    <origin xyz="-0.092 0.0 0.091" rpy="0 0 0" />
+    <parent link="$(arg prefix)base_link"/>
+    <child link="$(arg prefix)link1"/>
+    <origin xyz="-0.092 0.0 0.091" rpy="0 0 0"/>
   </joint>
   <xacro:open_manipulator_x prefix="$(arg prefix)" />
@@ -31,5 +31,5 @@
     name="TurtleBot3ManipulationSystem" prefix="$(arg prefix)" use_sim="$(arg use_sim)"
     use_fake_hardware="$(arg use_fake_hardware)"
-    fake_sensor_commands="$(arg fake_sensor_commands)" />
+    fake_sensor_commands="$(arg fake_sensor_commands)"/>
   <gazebo>
     <plugin filename="gz_ros2_control-system" name="gz_ros2_control::GazeboSimROS2ControlPlugin">
@@ -37,7 +37,4 @@
       <robot_param_node>robot_state_publisher</robot_param_node>
       <parameters>$(find turtlebot3_manipulation_bringup)/config/hardware_controller_manager.yaml</parameters>
-      <!-- <ros>
-      <remapping>/diff_drive_controller/cmd_vel:=/cmd_vel</remapping>
-      </ros> -->
     </plugin>
   </gazebo>

File: turtlebot3_manipulation_description/urdf/turtlebot3_waffle_pi.urdf.xacro (robot description, xacro)
@@ -38,5 +38,5 @@
                iyy="8.6195418e-03" iyz="-3.5422299e-06"
                izz="1.4612727e-02" />
-    </inertial>07
+    </inertial>
   </link>
   <joint name="${prefix}wheel_left_joint" type="continuous">
