Commit message: fixed inertial tensors and can navigate with known map. SLAM not working well

File: turtlebot3_manipulation_description/urdf/turtlebot3_waffle_pi.urdf.xacro (robot description, xacro)
@@ -18,5 +18,6 @@
   <link name="${prefix}base_link">
     <visual>
-      <origin xyz="-0.064 0 0.0" rpy="0 0 0"/>
+      <!-- <origin xyz="-0.064 0 0.0" rpy="0 0 0"/> -->
+      <origin xyz="0 0 0.0" rpy="0 0 0"/>
       <geometry>
         <mesh filename="${meshes_file_direction}/base.stl" scale="0.001 0.001 0.001"/>
@@ -25,5 +26,6 @@
     </visual>
     <collision>
-      <origin xyz="-0.064 0 0.047" rpy="0 0 0"/>
+      <!-- <origin xyz="-0.064 0 0.047" rpy="0 0 0"/> -->
+      <origin xyz="0.0 0 0.047" rpy="0 0 0"/>
       <geometry>
         <box size="0.266 0.266 0.094"/>
@@ -31,15 +33,15 @@
     </collision>
     <inertial>
-      <origin xyz="0 0 0" rpy="0 0 0"/>
+      <origin xyz="0 0 0" rpy="0 -0.155 0"/>
       <mass value="1.3729096e+00"/>
       <inertia ixx="8.7002718e-03" ixy="-4.7576583e-05" ixz="1.1160499e-04"
                iyy="8.6195418e-03" iyz="-3.5422299e-06"
                izz="1.4612727e-02" />
-    </inertial>
+    </inertial>07
   </link>
   <joint name="${prefix}wheel_left_joint" type="continuous">
     <parent link="${prefix}base_link"/>
     <child link="${prefix}wheel_left_link"/>
-    <origin xyz="0.0 0.144 0.023" rpy="-1.57 0 0"/>
+    <origin xyz="0.064 0.144 0.023" rpy="-1.57 0 0"/>
     <axis xyz="0 0 1"/>
   </joint>
@@ -69,5 +71,5 @@
     <parent link="${prefix}base_link"/>
     <child link="${prefix}wheel_right_link"/>
-    <origin xyz="0.0 -0.144 0.023" rpy="-1.57 0 0"/>
+    <origin xyz="0.064 -0.144 0.023" rpy="-1.57 0 0"/>
     <axis xyz="0 0 1"/>
   </joint>
@@ -101,5 +103,5 @@
   <link name="${prefix}caster_back_right_link">
     <collision>
-      <origin xyz="0 0.001 0" rpy="0 0 0"/>
+      <origin xyz="0.064 0.001 0" rpy="0 0 0"/>
       <geometry>
         <box size="0.030 0.009 0.020"/>
@@ -121,5 +123,5 @@
   <link name="${prefix}caster_back_left_link">
     <collision>
-      <origin xyz="0 0.001 0" rpy="0 0 0"/>
+      <origin xyz="0.064 0.001 0" rpy="0 0 0"/>
       <geometry>
         <box size="0.030 0.009 0.020"/>

Commit message: fixed robot inertial model and base link. again

File: turtlebot3_manipulation_description/urdf/turtlebot3_waffle_pi.urdf.xacro (robot description, xacro)
@@ -19,5 +19,5 @@
     <visual>
       <!-- <origin xyz="-0.064 0 0.0" rpy="0 0 0"/> -->
-      <origin xyz="0 0 0.0" rpy="0 0 0"/>
+      <origin xyz="-0.064 0 0.0" rpy="0 0 0"/>
       <geometry>
         <mesh filename="${meshes_file_direction}/base.stl" scale="0.001 0.001 0.001"/>
@@ -27,5 +27,5 @@
     <collision>
       <!-- <origin xyz="-0.064 0 0.047" rpy="0 0 0"/> -->
-      <origin xyz="0.0 0 0.047" rpy="0 0 0"/>
+      <origin xyz="-0.064 0 0.047" rpy="0 0 0"/>
       <geometry>
         <box size="0.266 0.266 0.094"/>
@@ -33,8 +33,12 @@
     </collision>
     <inertial>
-      <origin xyz="0 0 0" rpy="0 -0.155 0"/>
+      <!-- <origin xyz="-0.064 0 0" rpy="0 -0.155 0"/> -->
+      <origin xyz="-0.064 0 0" rpy="0 0 0"/>
       <mass value="1.3729096e+00"/>
-      <inertia ixx="8.7002718e-03" ixy="-4.7576583e-05" ixz="1.1160499e-04"
+      <!-- <inertia ixx="8.7002718e-03" ixy="-4.7576583e-05" ixz="1.1160499e-04"
                iyy="8.6195418e-03" iyz="-3.5422299e-06"
+               izz="1.4612727e-02" /> -->
+      <inertia ixx="8.7002718e-03" ixy="0.0" ixz="0.0"
+               iyy="8.6195418e-03" iyz="0.0"
                izz="1.4612727e-02" />
     </inertial>
@@ -43,5 +47,5 @@
     <parent link="${prefix}base_link"/>
     <child link="${prefix}wheel_left_link"/>
-    <origin xyz="0.064 0.144 0.023" rpy="-1.57 0 0"/>
+    <origin xyz="0.0 0.144 0.023" rpy="-1.57 0 0"/>
     <axis xyz="0 0 1"/>
   </joint>
@@ -71,5 +75,5 @@
     <parent link="${prefix}base_link"/>
     <child link="${prefix}wheel_right_link"/>
-    <origin xyz="0.064 -0.144 0.023" rpy="-1.57 0 0"/>
+    <origin xyz="0.0 -0.144 0.023" rpy="-1.57 0 0"/>
     <axis xyz="0 0 1"/>
   </joint>

Commit message: second attempt to re-enable simulation world

File: turtlebot3_manipulation_description/urdf/turtlebot3_waffle_pi.urdf.xacro (robot description, xacro)
@@ -31,8 +31,8 @@
     </collision>
     <inertial>
-      <origin xyz="0 0 0" rpy="0 0 0"/>
+      <origin xyz="-0.064 0 0" rpy="0 0 0"/>
       <mass value="1.3729096e+00"/>
-      <inertia ixx="8.7002718e-03" ixy="-4.7576583e-05" ixz="1.1160499e-04"
-               iyy="8.6195418e-03" iyz="-3.5422299e-06"
+      <inertia ixx="8.7002718e-03" ixy="0.0" ixz="0.0"
+               iyy="8.6195418e-03" iyz="0.0"
                izz="1.4612727e-02" />
     </inertial>
@@ -97,9 +97,9 @@
     <parent link="${prefix}base_link"/>
     <child link="${prefix}caster_back_right_link"/>
-    <origin xyz="-0.177 -0.064 -0.004" rpy="-1.57 0 0"/>
+    <origin xyz="-0.237 -0.064 -0.004" rpy="-1.57 0 0"/>
   </joint>
   <link name="${prefix}caster_back_right_link">
     <collision>
-      <origin xyz="0 0.001 0" rpy="0 0 0"/>
+      <origin xyz="0.064 0.001 0" rpy="0 0 0"/>
       <geometry>
         <box size="0.030 0.009 0.020"/>
@@ -117,9 +117,9 @@
     <parent link="${prefix}base_link"/>
     <child link="${prefix}caster_back_left_link"/>
-    <origin xyz="-0.177 0.064 -0.004" rpy="-1.57 0 0"/>
+    <origin xyz="-0.237 0.064 -0.004" rpy="-1.57 0 0"/>
   </joint>
   <link name="${prefix}caster_back_left_link">
     <collision>
-      <origin xyz="0 0.001 0" rpy="0 0 0"/>
+      <origin xyz="0.064 0.001 0" rpy="0 0 0"/>
       <geometry>
         <box size="0.030 0.009 0.020"/>
