Commit message: added twist mux and cleaned up joystick control

File: turtlebot3_manipulation_description/ros2_control/turtlebot3_manipulation_system.ros2_control.xacro (robot description, xacro)
@@ -6,5 +6,6 @@
 -->
 <robot xmlns:xacro="http://www.ros.org/wiki/xacro">
-  <xacro:macro name="turtlebot3_manipulation_system" params="name prefix use_sim:=^|false use_fake_hardware:=^|false fake_sensor_commands:=^|false">
+  <xacro:macro name="turtlebot3_manipulation_system"
+    params="name prefix use_sim:=^|false use_fake_hardware:=^|false fake_sensor_commands:=^|false">
     <ros2_control name="${name}" type="system">
       <xacro:if value="$(arg use_sim)">

File: turtlebot3_manipulation_description/urdf/turtlebot3_manipulation.urdf.xacro (robot description, xacro)
@@ -9,13 +9,18 @@
   <xacro:include filename="$(find turtlebot3_manipulation_description)/gazebo/materials.xacro" />
   <!-- Include TurtleBot3 Waffle Pi urdf macro -->
-  <xacro:include filename="$(find turtlebot3_manipulation_description)/urdf/turtlebot3_waffle_pi.urdf.xacro" />
+  <xacro:include
+    filename="$(find turtlebot3_manipulation_description)/urdf/turtlebot3_waffle_pi.urdf.xacro" />
   <!-- Include TurtleBot3 Waffle Pi gazebo macro -->
-  <xacro:include filename="$(find turtlebot3_manipulation_description)/gazebo/turtlebot3_waffle_pi.gazebo.xacro" />
+  <xacro:include
+    filename="$(find turtlebot3_manipulation_description)/gazebo/turtlebot3_waffle_pi.gazebo.xacro" />
   <!-- Include OpenManipulator-X urdf macro -->
-  <xacro:include filename="$(find turtlebot3_manipulation_description)/urdf/open_manipulator_x.urdf.xacro" />
+  <xacro:include
+    filename="$(find turtlebot3_manipulation_description)/urdf/open_manipulator_x.urdf.xacro" />
   <!-- Include OpenManipulator-X gazebo macro -->
-  <xacro:include filename="$(find turtlebot3_manipulation_description)/gazebo/open_manipulator_x.gazebo.xacro" />
+  <xacro:include
+    filename="$(find turtlebot3_manipulation_description)/gazebo/open_manipulator_x.gazebo.xacro" />
   <!-- Include TurtleBot3 Manipulation ros2 control macro -->
-  <xacro:include filename="$(find turtlebot3_manipulation_description)/ros2_control/turtlebot3_manipulation_system.ros2_control.xacro" />
+  <xacro:include
+    filename="$(find turtlebot3_manipulation_description)/ros2_control/turtlebot3_manipulation_system.ros2_control.xacro" />
   <xacro:turtlebot3_waffle_pi prefix="$(arg prefix)" />
   <xacro:turtlebot3_waffle_pi_gazebo prefix="$(arg prefix)" />
@@ -37,4 +42,7 @@
       <robot_param_node>robot_state_publisher</robot_param_node>
       <parameters>$(find turtlebot3_manipulation_bringup)/config/hardware_controller_manager.yaml</parameters>
+      <!-- <ros>
+      <remapping>/diff_drive_controller/cmd_vel:=/cmd_vel</remapping>
+      </ros> -->
     </plugin>
   </gazebo>

Commit message: synch with wpjazzy sim changes

File: turtlebot3_manipulation_description/ros2_control/turtlebot3_manipulation_system.ros2_control.xacro (robot description, xacro)
@@ -6,9 +6,10 @@
 -->
 <robot xmlns:xacro="http://www.ros.org/wiki/xacro">
-  <xacro:macro name="turtlebot3_manipulation_system" params="name prefix use_sim:=^|false use_fake_hardware:=^|false fake_sensor_commands:=^|false">
+  <xacro:macro name="turtlebot3_manipulation_system"
+    params="name prefix use_sim:=^|false use_fake_hardware:=^|false fake_sensor_commands:=^|false">
     <ros2_control name="${name}" type="system">
       <xacro:if value="$(arg use_sim)">
         <hardware>
-          <plugin>gazebo_ros2_control/GazeboSystem</plugin>
+          <plugin>gz_ros2_control/GazeboSimSystem</plugin>
         </hardware>
       </xacro:if>
@@ -165,8 +166,8 @@
         <param name="mimic">gripper_left_joint</param>
         <param name="multiplier">1</param>
-        <command_interface name="position">
+        <!-- <command_interface name="position">
           <param name="min">-0.010</param>
           <param name="max">0.019</param>
-        </command_interface>
+        </command_interface> -->
         <state_interface name="position">
           <param name="initial_value">0.0</param>

File: turtlebot3_manipulation_description/urdf/turtlebot3_manipulation.urdf.xacro (robot description, xacro)
@@ -33,6 +33,8 @@
     fake_sensor_commands="$(arg fake_sensor_commands)"/>
   <gazebo>
-    <plugin name="gazebo_ros2_control" filename="libgazebo_ros2_control.so">
-      <parameters>$(find turtlebot3_manipulation_bringup)/config/gazebo_controller_manager.yaml</parameters>
+    <plugin filename="gz_ros2_control-system" name="gz_ros2_control::GazeboSimROS2ControlPlugin">
+      <robot_param>robot_description</robot_param>
+      <robot_param_node>robot_state_publisher</robot_param_node>
+      <parameters>$(find turtlebot3_manipulation_bringup)/config/hardware_controller_manager.yaml</parameters>
     </plugin>
   </gazebo>

File: turtlebot3_manipulation_description/urdf/turtlebot3_waffle_pi.urdf.xacro (robot description, xacro)
@@ -18,4 +18,5 @@
   <link name="${prefix}base_link">
     <visual>
+      <!-- <origin xyz="-0.064 0 0.0" rpy="0 0 0"/> -->
       <origin xyz="-0.064 0 0.0" rpy="0 0 0"/>
       <geometry>
@@ -25,4 +26,5 @@
     </visual>
     <collision>
+      <!-- <origin xyz="-0.064 0 0.047" rpy="0 0 0"/> -->
       <origin xyz="-0.064 0 0.047" rpy="0 0 0"/>
       <geometry>
@@ -31,8 +33,12 @@
     </collision>
     <inertial>
-      <origin xyz="0 0 0" rpy="0 0 0"/>
+      <!-- <origin xyz="-0.064 0 0" rpy="0 -0.155 0"/> -->
+      <origin xyz="-0.064 0 0" rpy="0 0 0"/>
       <mass value="1.3729096e+00"/>
-      <inertia ixx="8.7002718e-03" ixy="-4.7576583e-05" ixz="1.1160499e-04"
+      <!-- <inertia ixx="8.7002718e-03" ixy="-4.7576583e-05" ixz="1.1160499e-04"
                iyy="8.6195418e-03" iyz="-3.5422299e-06"
+               izz="1.4612727e-02" /> -->
+      <inertia ixx="8.7002718e-03" ixy="0.0" ixz="0.0"
+               iyy="8.6195418e-03" iyz="0.0"
                izz="1.4612727e-02" />
     </inertial>
@@ -101,5 +107,5 @@
   <link name="${prefix}caster_back_right_link">
     <collision>
-      <origin xyz="0 0.001 0" rpy="0 0 0"/>
+      <origin xyz="0.064 0.001 0" rpy="0 0 0"/>
       <geometry>
         <box size="0.030 0.009 0.020"/>
@@ -121,5 +127,5 @@
   <link name="${prefix}caster_back_left_link">
     <collision>
-      <origin xyz="0 0.001 0" rpy="0 0 0"/>
+      <origin xyz="0.064 0.001 0" rpy="0 0 0"/>
       <geometry>
         <box size="0.030 0.009 0.020"/>

Commit message: fixed the lower limit for the gripper to 0.02

File: turtlebot3_manipulation_description/ros2_control/turtlebot3_manipulation_system.ros2_control.xacro (robot description, xacro)
@@ -152,5 +152,5 @@
       <joint name="${prefix}gripper_left_joint">
         <command_interface name="position">
-          <param name="min">-0.010</param>
+          <param name="min">-0.020</param>
           <param name="max">0.019</param>
         </command_interface>

File: turtlebot3_manipulation_description/urdf/open_manipulator_x.urdf.xacro (robot description, xacro)
@@ -157,5 +157,5 @@
       <origin xyz="0.0817 0.021 0.0" rpy="0 0 0"/>
       <axis xyz="0 1 0"/>
-      <limit velocity="4.8" effort="1" lower="-0.010" upper="0.019" />
+      <limit velocity="4.8" effort="1" lower="-0.020" upper="0.019" />
       <dynamics damping="0.1"/>
     </joint>
@@ -192,5 +192,5 @@
       <origin xyz="0.0817 -0.021 0" rpy="0 0 0"/>
       <axis xyz="0 -1 0"/>
-      <limit velocity="4.8" effort="1" lower="-0.010" upper="0.019" />
+      <limit velocity="4.8" effort="1" lower="-0.020" upper="0.019" />
       <mimic joint="${prefix}gripper_left_joint" multiplier="1"/>
       <dynamics damping="0.1"/>

File: turtlebot3_manipulation_description/urdf/tbotomx.urdf (robot description, URDF)
Before this commit: robot turtlebot3_manipulation, 20 links, 19 joints
Joints:
- joint gripper_left_joint: limit lower=-0.010 upper=0.019 effort=1 velocity=4.8 -> lower=-0.020 upper=0.019 effort=1 velocity=4.8
- joint gripper_right_joint: limit lower=-0.010 upper=0.019 effort=1 velocity=4.8 -> lower=-0.020 upper=0.019 effort=1 velocity=4.8

Commit message: first attempt to re-enable simulation world

File: turtlebot3_manipulation_description/ros2_control/turtlebot3_manipulation_system.ros2_control.xacro (robot description, xacro)
@@ -6,9 +6,10 @@
 -->
 <robot xmlns:xacro="http://www.ros.org/wiki/xacro">
-  <xacro:macro name="turtlebot3_manipulation_system" params="name prefix use_sim:=^|false use_fake_hardware:=^|false fake_sensor_commands:=^|false">
+  <xacro:macro name="turtlebot3_manipulation_system"
+    params="name prefix use_sim:=^|false use_fake_hardware:=^|false fake_sensor_commands:=^|false">
     <ros2_control name="${name}" type="system">
       <xacro:if value="$(arg use_sim)">
         <hardware>
-          <plugin>gazebo_ros2_control/GazeboSystem</plugin>
+          <plugin>gz_ros2_control/GazeboSimSystem</plugin>
         </hardware>
       </xacro:if>

Commit message: adjusted gripper limits to observed limits

File: turtlebot3_manipulation_description/ros2_control/turtlebot3_manipulation_system.ros2_control.xacro (robot description, xacro)
@@ -153,6 +153,6 @@
       <joint name="${prefix}gripper_left_joint">
         <command_interface name="position">
-          <param name="min">-0.020</param>
-          <param name="max">0.019</param>
+          <param name="min">-0.014</param>
+          <param name="max">0.018</param>
         </command_interface>
         <state_interface name="position">

File: turtlebot3_manipulation_description/urdf/open_manipulator_x.urdf.xacro (robot description, xacro)
@@ -157,5 +157,5 @@
       <origin xyz="0.0817 0.021 0.0" rpy="0 0 0" />
       <axis xyz="0 1 0" />
-      <limit velocity="4.8" effort="1" lower="-0.020" upper="0.019" />
+      <limit velocity="4.8" effort="1" lower="-0.014" upper="0.018" />
       <dynamics damping="0.1" />
     </joint>
@@ -192,5 +192,5 @@
       <origin xyz="0.0817 -0.021 0" rpy="0 0 0" />
       <axis xyz="0 -1 0" />
-      <limit velocity="4.8" effort="1" lower="-0.020" upper="0.019" />
+      <limit velocity="4.8" effort="1" lower="-0.014" upper="0.018" />
       <mimic joint="${prefix}gripper_left_joint" multiplier="1" />
       <dynamics damping="0.1" />

File: turtlebot3_manipulation_description/urdf/tbotomx.urdf (robot description, URDF)
Before this commit: robot turtlebot3_manipulation, 20 links, 19 joints
Joints:
- joint gripper_left_joint: limit lower=-0.020 upper=0.019 effort=1 velocity=4.8 -> lower=-0.014 upper=0.018 effort=1 velocity=4.8
- joint gripper_right_joint: limit lower=-0.020 upper=0.019 effort=1 velocity=4.8 -> lower=-0.014 upper=0.018 effort=1 velocity=4.8
